File: kicad/oculink_m2.kicad_sch (KiCad schematic)
At the start: 18 parts, among them J1 G14A42121B12HR

Commit message: Temporary mockup of adtlink adapter
Parts:
- removed D1: BAT64-02W, Diode_SMD:D_SOD-523, symbol Device:D_Schottky
- removed TP1: TP_EXT_CWAKE, TestPoint:TestPoint_Pad_D1.0mm, symbol Connector:TestPoint
- removed TP10: TP_GND_1, TestPoint:TestPoint_Pad_D1.0mm, symbol Connector:TestPoint
- removed TP2: TP_EXT_5V_1, TestPoint:TestPoint_Pad_D1.0mm, symbol Connector:TestPoint
- removed TP3: TP_EXT_3.3V, TestPoint:TestPoint_Pad_D1.0mm, symbol Connector:TestPoint
- removed TP4: TP_EXT_5V_2, TestPoint:TestPoint_Pad_D1.0mm, symbol Connector:TestPoint
- removed TP5: TP_M2_LED, TestPoint:TestPoint_Pad_D1.0mm, symbol Connector:TestPoint
- removed TP6: TP_M2_PEWAKE, TestPoint:TestPoint_Pad_D1.0mm, symbol Connector:TestPoint
- removed TP7: TP_M2_DEVSLP, TestPoint:TestPoint_Pad_D1.0mm, symbol Connector:TestPoint
- removed TP8: TP_M2_SUSCLK, TestPoint:TestPoint_Pad_D1.0mm, symbol Connector:TestPoint
- added H1: M2_MOUNT, custom_edge_connector:m2_ground_hole, symbol Mechanical:MountingHole_Pad
- added JP3: JMP_PEWAKE, Jumper:SolderJumper-2_P1.3mm_Open_RoundedPad1.0x1.5mm, symbol Jumper:SolderJumper_2_Open
- added JP4: JMP_CLKREQ, Jumper:SolderJumper-2_P1.3mm_Open_RoundedPad1.0x1.5mm, symbol Jumper:SolderJumper_2_Open
- added JP5: JMP_CWAKE, Jumper:SolderJumper-2_P1.3mm_Open_RoundedPad1.0x1.5mm, symbol Jumper:SolderJumper_2_Open
- J1: footprint amphenol_oculink:AMPHENOL_G14A42121B12HR -> amphenol_oculink:AMPHENOL_G14A421211112HR; symbol G14A42121B12HR:G14A42121B12HR -> G14A421211112HR:G14A421211112HR; MAXIMUM_PACKAGE_HEIGHT 3.9mm -> 3.92mm; PARTREV D -> A
- JP1: value SolderJumper_2_Open -> JMP_PEDET
- JP2: value SolderJumper_2_Open -> JMP_3.3V_EXT
Connections:
- net CLKREQ: now also J1.B13 (CPRSNT), JP4.2 (B)
- net GND: now also H1.1, JP3.1 (A), JP4.1 (A)
- net PEWAKE: now reaches E1.54 (~{PEWAKE})
- net PEWAKE: now also JP3.2 (B), JP5.1 (A)
- net at J1.A10 (CWAKE): now also JP5.2 (B)
- no-connect marks 21 -> 26
Other:
- note removed: "LCSC Part #: C475624"
- moved on the sheet: JP1, TP9

Commit message: Preliminary routing of pcie lanes over bottleneck in pcb
Connections:
- net SMB_CLOCK: now reaches E1.40 (SMB_CLOCK)
- net SMB_CLOCK: now also J1.B9 (CLOCK)
- net SMB_DATA: now reaches E1.42 (SMB_DATA)
- net SMB_DATA: now also J1.B10 (DATA)
- no-connect marks 26 -> 22
Other:
- moved on the sheet: JP3, JP4
Changed lines of the file:
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@@
 	)
 	(junction
-		(at 43.18 106.68)
+		(at 36.83 106.68)
 		(diameter 0)
 		(color 0 0 0 0)
@@
 	)
 	(junction
-		(at 48.26 85.09)
+		(at 41.91 85.09)
 		(diameter 0)
 		(color 0 0 0 0)
@@
 	)
 	(junction
-		(at 38.1 87.63)
+		(at 31.75 87.63)
 		(diameter 0)
 		(color 0 0 0 0)
@@
 	)
 	(no_connect
-		(at 68.58 100.33)
-	)
-	(no_connect
 		(at 68.58 123.19)
 	)
@@
 	)
 	(no_connect
-		(at 199.39 106.68)
-	)
-	(no_connect
 		(at 68.58 118.11)
 	)
@@
 	)
 	(no_connect
-		(at 199.39 104.14)
-	)
-	(no_connect
 		(at 68.58 82.55)
 	)
@@
 	)
 	(no_connect
-		(at 68.58 102.87)
-	)
-	(no_connect
 		(at 68.58 67.31)
 	)
@@
 	(wire
 		(pts
-			(xy 38.1 100.33) (xy 38.1 106.68)
+			(xy 31.75 100.33) (xy 31.75 106.68)
 		)
 		(stroke
@@
 	(wire
 		(pts
-			(xy 38.1 87.63) (xy 68.58 87.63)
+			(xy 31.75 87.63) (xy 68.58 87.63)
 		)
 		(stroke
@@
 	(wire
 		(pts
+			(xy 60.96 102.87) (xy 68.58 102.87)
+		)
+		(stroke
+			(width 0)
+			(type default)
+		)
+	)
+	(wire
+		(pts
 			(xy 139.7 39.37) (xy 146.05 39.37)
 		)
@@
 	(wire
 		(pts
-			(xy 38.1 106.68) (xy 43.18 106.68)
+			(xy 31.75 106.68) (xy 36.83 106.68)
 		)
 		(stroke
@@
 	(wire
 		(pts
-			(xy 48.26 92.71) (xy 48.26 85.09)
+			(xy 41.91 92.71) (xy 41.91 85.09)
 		)
 		(stroke
@@
 	(wire
 		(pts
+			(xy 199.39 106.68) (xy 207.01 106.68)
+		)
+		(stroke
+			(width 0)
+			(type default)
+		)
+	)
+	(wire
+		(pts
 			(xy 66.04 64.77) (xy 68.58 64.77)
 		)
@@
 	(wire
 		(pts
-			(xy 26.67 85.09) (xy 48.26 85.09)
+			(xy 26.67 85.09) (xy 41.91 85.09)
 		)
 		(stroke
@@
 	(wire
 		(pts
-			(xy 48.26 85.09) (xy 68.58 85.09)
+			(xy 41.91 85.09) (xy 68.58 85.09)
 		)
 		(stroke
@@
 	(wire
 		(pts
+			(xy 199.39 104.14) (xy 207.01 104.14)
+		)
+		(stroke
+			(width 0)
+			(type default)
+		)
+	)
+	(wire
+		(pts
 			(xy 146.05 52.07) (xy 157.48 52.07)
 		)
@@
 	(wire
 		(pts
-			(xy 48.26 106.68) (xy 48.26 100.33)
+			(xy 41.91 106.68) (xy 41.91 100.33)
 		)
 		(stroke
@@
 	(wire
 		(pts
-			(xy 43.18 106.68) (xy 48.26 106.68)
+			(xy 36.83 106.68) (xy 41.91 106.68)
 		)
 		(stroke
@@
 	(wire
 		(pts
-			(xy 43.18 106.68) (xy 43.18 110.49)
+			(xy 36.83 106.68) (xy 36.83 110.49)
 		)
 		(stroke
@@
 	(wire
 		(pts
-			(xy 26.67 87.63) (xy 38.1 87.63)
+			(xy 26.67 87.63) (xy 31.75 87.63)
 		)
 		(stroke
@@
 	(wire
 		(pts
-			(xy 38.1 87.63) (xy 38.1 92.71)
+			(xy 31.75 87.63) (xy 31.75 92.71)
 		)
 		(stroke
@@
 	(wire
 		(pts
+			(xy 60.96 100.33) (xy 68.58 100.33)
+		)
+		(stroke
+			(width 0)
+			(type default)
+		)
+	)
+	(wire
+		(pts
 			(xy 66.04 59.69) (xy 66.04 62.23)
 		)
@@
 		)
 	)
+	(global_label "SMB_DATA"
+		(shape output)
+		(at 207.01 106.68 0)
+		(fields_autoplaced yes)
+		(effects
+			(font
+				(size 1.27 1.27)
+			)
+			(justify left)
+		)
+		(property "Intersheetrefs" "${INTERSHEET_REFS}"
+			(at 219.3085 106.68 0)
+			(effects
+				(font
+					(size 1.27 1.27)
+				)
+				(justify left)
+				(hide yes)
+			)
+		)
+	)
 	(global_label "RX1-"
 		(shape input)
@@
 		)
 	)
+	(global_label "SMB_DATA"
+		(shape input)
+		(at 60.96 100.33 180)
+		(fields_autoplaced yes)
+		(effects
+			(font
+				(size 1.27 1.27)
+			)
+			(justify right)
+		)
+		(property "Intersheetrefs" "${INTERSHEET_REFS}"
+			(at 48.6615 100.33 0)
+			(effects
+				(font
+					(size 1.27 1.27)
+				)
+				(justify right)
+				(hide yes)
+			)
+		)
+	)
 	(global_label "3.3V_OPT"
 		(shape output)
@@
 		)
 	)
+	(global_label "SMB_CLOCK"
+		(shape input)
+		(at 60.96 102.87 180)
+		(fields_autoplaced yes)
+		(effects
+			(font
+				(size 1.27 1.27)
+			)
+			(justify right)
+		)
+		(property "Intersheetrefs" "${INTERSHEET_REFS}"
+			(at 46.9077 102.87 0)
+			(effects
+				(font
+					(size 1.27 1.27)
+				)
+				(justify right)
+				(hide yes)
+			)
+		)
+	)
 	(global_label "RX3-"
 		(shape input)
@@
 		)
 	)
+	(global_label "SMB_CLOCK"
+		(shape output)
+		(at 207.01 104.14 0)
+		(fields_autoplaced yes)
+		(effects
+			(font
+				(size 1.27 1.27)
+			)
+			(justify left)
+		)
+		(property "Intersheetrefs" "${INTERSHEET_REFS}"
+			(at 221.0623 104.14 0)
+			(effects
+				(font
+					(size 1.27 1.27)
+				)
+				(justify left)
+				(hide yes)
+			)
+		)
+	)
 	(global_label "CLOCK+"
 		(shape output)
@@
 	(symbol
 		(lib_id "Jumper:SolderJumper_2_Open")
-		(at 38.1 96.52 90)
+		(at 31.75 96.52 90)
 		(unit 1)
 		(exclude_from_sim yes)
@@
 		(dnp no)
 		(property "Reference" "JP4"
-			(at 31.75 96.52 0)
+			(at 25.4 96.52 0)
 			(effects
 				(font
@@
 		)
 		(property "Value" "JMP_CLKREQ"
-			(at 34.798 96.266 0)
+			(at 28.448 96.266 0)
 			(effects
 				(font
@@
 		)
 		(property "Footprint" "Jumper:SolderJumper-2_P1.3mm_Open_RoundedPad1.0x1.5mm"
-			(at 38.1 96.52 0)
+			(at 31.75 96.52 0)
 			(effects
 				(font
@@
 		)
 		(property "Datasheet" "~"
-			(at 38.1 96.52 0)
+			(at 31.75 96.52 0)
 			(effects
 				(font
@@
 		)
 		(property "Description" "Solder Jumper, 2-pole, open"
-			(at 38.1 96.52 0)
+			(at 31.75 96.52 0)
 			(effects
 				(font
@@
 	(symbol
 		(lib_id "power:GND")
-		(at 43.18 110.49 0)
+		(at 36.83 110.49 0)
 		(unit 1)
 		(exclude_from_sim no)
@@
 		(dnp no)
 		(property "Reference" "#PWR07"
-			(at 43.18 116.84 0)
+			(at 36.83 116.84 0)
 			(effects
 				(font
@@
 		)
 		(property "Value" "GND"
-			(at 43.18 115.57 0)
+			(at 36.83 115.57 0)
 			(effects
 				(font
@@
 		)
 		(property "Footprint" ""
-			(at 43.18 110.49 0)
+			(at 36.83 110.49 0)
 			(effects
 				(font
@@
 		)
 		(property "Datasheet" ""
-			(at 43.18 110.49 0)
+			(at 36.83 110.49 0)
 			(effects
 				(font
@@
 		)
 		(property "Description" "Power symbol creates a global label with name \"GND\" , ground"
-			(at 43.18 110.49 0)
+			(at 36.83 110.49 0)
 			(effects
 				(font
@@
 	(symbol
 		(lib_id "Jumper:SolderJumper_2_Open")
-		(at 48.26 96.52 90)
+		(at 41.91 96.52 90)
 		(unit 1)
 		(exclude_from_sim yes)
@@
 		(dnp no)
 		(property "Reference" "JP3"
-			(at 41.91 96.52 0)
+			(at 35.56 96.52 0)
 			(effects
 				(font
@@
 		)
 		(property "Value" "JMP_PEWAKE"
-			(at 44.958 96.266 0)
+			(at 38.608 96.266 0)
 			(effects
 				(font
@@
 		)
 		(property "Footprint" "Jumper:SolderJumper-2_P1.3mm_Open_RoundedPad1.0x1.5mm"
-			(at 48.26 96.52 0)
+			(at 41.91 96.52 0)
 			(effects
 				(font
@@
 		)
 		(property "Datasheet" "~"
-			(at 48.26 96.52 0)
+			(at 41.91 96.52 0)
 			(effects
 				(font
@@
 		)
 		(property "Description" "Solder Jumper, 2-pole, open"
-			(at 48.26 96.52 0)
+			(at 41.91 96.52 0)
 			(effects
 				(font

Commit message: Finished prototype of potentially ready adapter
Parts:
- removed JP1: JMP_PEDET, Jumper:SolderJumper-2_P1.3mm_Open_RoundedPad1.0x1.5mm, symbol Jumper:SolderJumper_2_Open
- removed JP3: JMP_PEWAKE, Jumper:SolderJumper-2_P1.3mm_Open_RoundedPad1.0x1.5mm, symbol Jumper:SolderJumper_2_Open
- removed JP4: JMP_CLKREQ, Jumper:SolderJumper-2_P1.3mm_Open_RoundedPad1.0x1.5mm, symbol Jumper:SolderJumper_2_Open
- removed JP5: JMP_CWAKE, Jumper:SolderJumper-2_P1.3mm_Open_RoundedPad1.0x1.5mm, symbol Jumper:SolderJumper_2_Open
- added C4, C5: 100n, Capacitor_SMD:C_0402_1005Metric, symbol Device:C
- added JP1: JMP_PEDET, custom_edge_connector:3pin_4state_jumper, symbol Jumper:SolderJumper_3_Open
- added JP3: JMP_PEWAKE, custom_edge_connector:3pin_4state_jumper, symbol Jumper:SolderJumper_3_Open
- added TP1: TP_GND_1, TestPoint:TestPoint_Pad_D1.0mm, symbol Connector:TestPoint
Connections:
- net +3.3V: now also C4.1, C5.1
- net 3.3V_OPT: no longer J1.A1 (3.3V)
- net GND: now also C4.2, C5.2, JP1.2 (C), JP3.2 (C), TP1.1
- net PEDET: now also JP1.1 (A)
- net PEWAKE: now also JP3.1 (A)
- net PEDET_EXT: now reaches J1.A9 (RESERVED)
- net PEDET_EXT: now also JP1.3 (B)
- net PEWAKE_EXT: now reaches J1.A10 (CWAKE)
- net PEWAKE_EXT: now also JP3.3 (B)
- net SMB_CLOCK renamed SMB+
- net SMB+: now also E1.42 (SMB_DATA); no longer E1.40 (SMB_CLOCK)
- net SMB_DATA renamed SMB-
- net SMB-: now also E1.40 (SMB_CLOCK); no longer E1.42 (SMB_DATA)
- no-connect marks 22 -> 23

Commit message: Swapped SMB pair to connect clock/data correctly
Parts:
- J1: value G14A42121B12HR -> G14A421211112HR
Connections:
- net SMB+: now also J1.B10 (DATA); no longer J1.B9 (CLOCK)
- net SMB-: now also J1.B9 (CLOCK); no longer J1.B10 (DATA)

Commit message: Added working copy of gpdwin vertical adapter to confirm correct pinout
Parts:
- removed C1, C2, C3, C4, C5: 100n, Capacitor_SMD:C_0402_1005Metric, symbol Device:C
- removed JP1: JMP_PEDET, custom_edge_connector:3pin_4state_jumper, symbol Jumper:SolderJumper_3_Open
- removed JP2: JMP_3.3V_EXT, Jumper:SolderJumper-2_P1.3mm_Open_RoundedPad1.0x1.5mm, symbol Jumper:SolderJumper_2_Open
- removed JP3: JMP_PEWAKE, custom_edge_connector:3pin_4state_jumper, symbol Jumper:SolderJumper_3_Open
- J1: footprint amphenol_oculink:AMPHENOL_G14A421211112HR -> amphenol_oculink:AMPHENOL_G14A42211612HR; symbol G14A421211112HR:G14A421211112HR -> G14A42211612HR:G14A42211612HR; MAXIMUM_PACKAGE_HEIGHT 3.92mm -> 6.66 mm; PARTREV A -> F
Connections:
- net PEDET_EXT is gone; now on net PEWAKE: J1.A9 (RESERVED)
- net PEWAKE_EXT is gone; now on net GND: J1.A10 (CWAKE)
- net +3.3V: now also J1.B20 (GND)
- net CLKREQ: now also J1.B12 (PERST); no longer J1.B13 (CPRSNT)
- net CLOCK+: now also J1.A11 (GND); no longer J1.A12 (CLOCK+)
- net CLOCK-: now also J1.A12 (CLOCK+); no longer J1.A13 (CLOCK-)
- net GND: now also J1.A1 (3.3V), J1.A13 (CLOCK-), J1.A16 (PERn2), J1.A19 (PERn3), J1.A4 (PERn0), J1.A7 (PERn1), J1.B1 (5V), J1.B10 (DATA), J1.B13 (CPRSNT), J1.B16 (PETn2), J1.B19 (PETn3), J1.B4 (PETn0), J1.B7 (PETn1); no longer J1.A11 (GND), J1.A14 (GND), J1.A17 (GND), J1.A2 (GND), J1.A20 (GND), J1.A5 (GND), J1.A8 (GND), J1.B11 (GND), J1.B14 (GND), J1.B17 (GND), J1.B2 (GND), J1.B20 (GND), J1.B5 (GND), J1.B8 (GND), J1.SH3 (SHIELD_3), J1.SH4 (SHIELD_4)
- net PEDET: now also J1.A8 (GND)
- net PERST: now also J1.B11 (GND); no longer J1.B12 (PERST)
- net RX0+: now also J1.A2 (GND); no longer J1.A3 (PERp0)
- net RX0-: now also J1.A3 (PERp0); no longer J1.A4 (PERn0)
- net RX1+: now also J1.A5 (GND); no longer J1.A6 (PERp1)
- net RX1-: now also J1.A6 (PERp1); no longer J1.A7 (PERn1)
- net RX2+: now also J1.A14 (GND); no longer J1.A15 (PERp2)
- net RX2-: now also J1.A15 (PERp2); no longer J1.A16 (PERn2)
- net RX3+: now also J1.A17 (GND); no longer J1.A18 (PERp3)
- net RX3-: now also J1.A18 (PERp3); no longer J1.A19 (PERn3)
- net SMB+: now also J1.B9 (CLOCK); no longer J1.B10 (DATA)
- net SMB-: now also J1.B8 (GND); no longer J1.B9 (CLOCK)
- net TX0+: now also J1.B2 (GND); no longer J1.B3 (PETp0)
- net TX0-: now also J1.B3 (PETp0); no longer J1.B4 (PETn0)
- net TX1+: now also J1.B5 (GND); no longer J1.B6 (PETp1)
- net TX1-: now also J1.B6 (PETp1); no longer J1.B7 (PETn1)
- net TX2+: now also J1.B14 (GND); no longer J1.B15 (PETp2)
- net TX2-: now also J1.B15 (PETp2); no longer J1.B16 (PETn2)
- net TX3+: now also J1.B17 (GND); no longer J1.B18 (PETp3)
- net TX3-: now also J1.B18 (PETp3); no longer J1.B19 (PETn3)
- net 3.3V_OPT: no longer names the net of J1.B21 (3.3V)
Other:
- note removed: "LCSC Part #: C513772"
