File: kicad/oculink_m2.kicad_sch (KiCad schematic)
At the start: 13 parts, among them J1 G14A421211112HR

Commit message: Added additional mounting holes for adapter
Parts:
- added D1: Power LED, LED_SMD:LED_1206_3216Metric_Pad1.42x1.75mm_HandSolder, symbol Device:LED
- added H2: MOUNT_1, MountingHole:MountingHole_2.7mm, symbol Mechanical:MountingHole_Pad
- added H3: MOUNT_2, MountingHole:MountingHole_2.7mm, symbol Mechanical:MountingHole_Pad
- added R1: 100, Resistor_SMD:R_0603_1608Metric, symbol Device:R
Connections:
- net 3.3V_OPT: now also R1.1
- net GND: now also D1.1 (K)
- new net: D1.2 (A), R1.2
- no-connect marks 23 -> 25

Commit message: Fixed mounting holes
Parts:
- H2, H3: footprint MountingHole:MountingHole_2.7mm -> custom_edge_connector:secondary_mounting_hole; symbol Mechanical:MountingHole_Pad -> Mechanical:MountingHole
Connections:
- no-connect marks 25 -> 23
Changed lines of the file:
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@@
 	)
 	(no_connect
-		(at 250.19 48.26)
-	)
-	(no_connect
 		(at 68.58 82.55)
 	)
@@
 	)
 	(no_connect
-		(at 233.68 48.26)
-	)
-	(no_connect
 		(at 68.58 113.03)
 	)
@@
 	)
 	(symbol
-		(lib_id "Mechanical:MountingHole_Pad")
+		(lib_id "Mechanical:MountingHole")
 		(at 233.68 45.72 0)
 		(unit 1)
@@
 		(fields_autoplaced yes)
 		(property "Reference" "H2"
-			(at 236.22 43.1799 0)
+			(at 236.22 44.4499 0)
 			(effects
 				(font
@@
 		)
 		(property "Value" "MOUNT_1"
-			(at 236.22 45.7199 0)
+			(at 236.22 46.9899 0)
 			(effects
 				(font
@@
 			)
 		)
-		(property "Footprint" "MountingHole:MountingHole_2.7mm"
+		(property "Footprint" "custom_edge_connector:secondary_mounting_hole"
 			(at 233.68 45.72 0)
 			(effects
@@
 			)
 		)
-		(property "Description" "Mounting Hole with connection"
+		(property "Description" "Mounting Hole without connection"
 			(at 233.68 45.72 0)
 			(effects
@@
 			)
 		)
-		(pin "1"
-		)
 		(instances
 			(project ""
@@
 	)
 	(symbol
-		(lib_id "Mechanical:MountingHole_Pad")
+		(lib_id "Mechanical:MountingHole")
 		(at 250.19 45.72 0)
 		(unit 1)
@@
 		(fields_autoplaced yes)
 		(property "Reference" "H3"
-			(at 252.73 43.1799 0)
+			(at 252.73 44.4499 0)
 			(effects
 				(font
@@
 		)
 		(property "Value" "MOUNT_2"
-			(at 252.73 45.7199 0)
+			(at 252.73 46.9899 0)
 			(effects
 				(font
@@
 			)
 		)
-		(property "Footprint" "MountingHole:MountingHole_2.7mm"
+		(property "Footprint" "custom_edge_connector:secondary_mounting_hole"
 			(at 250.19 45.72 0)
 			(effects
@@
 			)
 		)
-		(property "Description" "Mounting Hole with connection"
+		(property "Description" "Mounting Hole without connection"
 			(at 250.19 45.72 0)
 			(effects
@@
 			)
 		)
-		(pin "1"
-		)
 		(instances

Commit message: Added bill of material and smd parts positioning scripts
Parts:
- C1, C2, C3, C4, C5: LCSC Part (none) -> C513772
- D1: LCSC Part (none) -> C434442
- E1, TP1, TP9: now left out of the parts list
- J1: LCSC Part (none) -> C5156927
- R1: LCSC Part (none) -> C22775
Changed lines of the file:
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@@
 		(unit 1)
 		(exclude_from_sim no)
-		(in_bom yes)
+		(in_bom no)
 		(on_board yes)
 		(dnp no)
@@
 			)
 		)
+		(property "LCSC Part" "C434442"
+			(at 247.65 88.9 90)
+			(effects
+				(font
+					(size 1.27 1.27)
+				)
+				(hide yes)
+			)
+		)
 		(pin "2"
 		)
@@
 		(unit 1)
 		(exclude_from_sim no)
-		(in_bom yes)
+		(in_bom no)
 		(on_board yes)
 		(dnp no)
@@
 		(unit 1)
 		(exclude_from_sim no)
-		(in_bom yes)
+		(in_bom no)
 		(on_board yes)
 		(dnp no)
@@
 			)
 		)
+		(property "LCSC Part" "C513772"
+			(at 134.62 45.72 0)
+			(effects
+				(font
+					(size 1.27 1.27)
+				)
+				(hide yes)
+			)
+		)
 		(pin "2"
 		)
@@
 			)
 		)
+		(property "LCSC Part" "C22775"
+			(at 247.65 78.74 0)
+			(effects
+				(font
+					(size 1.27 1.27)
+				)
+				(hide yes)
+			)
+		)
 		(pin "1"
 		)
@@
 			)
 		)
+		(property "LCSC Part" "C513772"
+			(at 186.69 45.72 0)
+			(effects
+				(font
+					(size 1.27 1.27)
+				)
+				(hide yes)
+			)
+		)
 		(pin "2"
 		)
@@
 			)
 		)
+		(property "LCSC Part" "C513772"
+			(at 146.05 45.72 0)
+			(effects
+				(font
+					(size 1.27 1.27)
+				)
+				(hide yes)
+			)
+		)
 		(pin "2"
 		)
@@
 			)
 		)
+		(property "LCSC Part" "C513772"
+			(at 123.19 45.72 0)
+			(effects
+				(font
+					(size 1.27 1.27)
+				)
+				(hide yes)
+			)
+		)
 		(pin "2"
 		)
@@
 			)
 		)
+		(property "LCSC Part" "C5156927"
+			(at 186.69 111.76 0)
+			(effects
+				(font
+					(size 1.27 1.27)
+				)
+				(hide yes)
+			)
+		)
 		(pin "A6"
 		)
@@
 			(at 157.48 45.72 0)
 			(effects
+				(font
+					(size 1.27 1.27)
+				)
+				(hide yes)
+			)
+		)
+		(property "LCSC Part" "C513772"
+			(at 157.48 45.72 0)
+			(effects

Commit message: Updated bom script and added in schottky diode on clkreq
Parts:
- added D2: D_Schottky, Diode_SMD:D_SOD-523, symbol Device:D_Schottky
Connections:
- net CLKREQ: now also D2.2 (A); no longer J1.B13 (CPRSNT)
- new net CLKREQ_EXT: D2.1 (K), J1.B13 (CPRSNT)
Other:
- note removed: "LCSC Part #: C513772"
Changed lines of the file:
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@@
 	(wire
 		(pts
-			(xy 199.39 114.3) (xy 207.01 114.3)
-		)
-		(stroke
-			(width 0)
-			(type default)
-		)
-	)
-	(wire
-		(pts
 			(xy 153.67 114.3) (xy 153.67 106.68)
 		)
@@
 	(wire
 		(pts
+			(xy 199.39 114.3) (xy 233.68 114.3)
+		)
+		(stroke
+			(width 0)
+			(type default)
+		)
+	)
+	(wire
+		(pts
 			(xy 171.45 116.84) (xy 171.45 124.46)
 		)
@@
 	(wire
 		(pts
+			(xy 241.3 114.3) (xy 245.11 114.3)
+		)
+		(stroke
+			(width 0)
+			(type default)
+		)
+	)
+	(wire
+		(pts
 			(xy 146.05 100.33) (xy 153.67 100.33)
 		)
@@
 		)
 	)
-	(text "LCSC Part #: C513772"
+	(text "Digikey Link"
 		(exclude_from_sim no)
-		(at 108.966 43.942 0)
+		(at 186.436 73.914 0)
 		(effects
 			(font
 				(size 1.27 1.27)
 			)
-			(href "https://www.lcsc.com/product-detail/Multilayer-Ceramic-Capacitors-MLCC---SMD-SMT_Samwha-Capacitor-Samwha-Capacitor-CS1005X7R104K500NR_C513772.html")
+			(href "https://www.digikey.com.au/en/products/detail/G14A421211112HR/664-G14A421211112HRCT-ND/17084317?curr=usd&utm_campaign=buynow&utm_medium=aggregator&utm_source=octopart")
 		)
 	)
-	(text "Digikey Link"
-		(exclude_from_sim no)
-		(at 186.436 73.914 0)
+	(label "CLKREQ_EXT"
+		(at 231.14 114.3 180)
+		(fields_autoplaced yes)
 		(effects
 			(font
 				(size 1.27 1.27)
 			)
-			(href "https://www.digikey.com.au/en/products/detail/G14A421211112HR/664-G14A421211112HRCT-ND/17084317?curr=usd&utm_campaign=buynow&utm_medium=aggregator&utm_source=octopart")
+			(justify right bottom)
 		)
 	)
@@
 		)
 	)
+	(global_label "CLKREQ"
+		(shape output)
+		(at 245.11 114.3 0)
+		(fields_autoplaced yes)
+		(effects
+			(font
+				(size 1.27 1.27)
+			)
+			(justify left)
+		)
+		(property "Intersheetrefs" "${INTERSHEET_REFS}"
+			(at 255.4128 114.3 0)
+			(effects
+				(font
+					(size 1.27 1.27)
+				)
+				(justify left)
+				(hide yes)
+			)
+		)
+	)
 	(global_label "TX2-"
 		(shape output)
@@
 		)
 	)
-	(global_label "CLKREQ"
-		(shape output)
-		(at 207.01 114.3 0)
-		(fields_autoplaced yes)
-		(effects
-			(font
-				(size 1.27 1.27)
-			)
-			(justify left)
-		)
-		(property "Intersheetrefs" "${INTERSHEET_REFS}"
-			(at 217.3128 114.3 0)
-			(effects
-				(font
-					(size 1.27 1.27)
-				)
-				(justify left)
-				(hide yes)
-			)
-		)
-	)
 	(global_label "RX2+"
 		(shape input)
@@
 					(unit 1)
 				)
+			)
+		)
+	)
+	(symbol
+		(lib_id "Device:D_Schottky")
+		(at 237.49 114.3 0)
+		(unit 1)
+		(exclude_from_sim no)
+		(in_bom yes)
+		(on_board yes)
+		(dnp no)
+		(fields_autoplaced yes)
+		(property "Reference" "D2"
+			(at 237.1725 107.95 0)
+			(effects
+				(font
+					(size 1.27 1.27)
+				)
+			)
+		)
+		(property "Value" "D_Schottky"
+			(at 237.1725 110.49 0)
+			(effects
+				(font
+					(size 1.27 1.27)
+				)
+			)
+		)
+		(property "Footprint" "Diode_SMD:D_SOD-523"
+			(at 237.49 114.3 0)
+			(effects
+				(font
+					(size 1.27 1.27)
+				)
+				(hide yes)
+			)
+		)
+		(property "Datasheet" "~"
+			(at 237.49 114.3 0)
+			(effects
+				(font
+					(size 1.27 1.27)
+				)
+				(hide yes)
+			)
+		)
+		(property "Description" "Schottky diode"
+			(at 237.49 114.3 0)
+			(effects
+				(font
+					(size 1.27 1.27)
+				)
+				(hide yes)
+			)
+		)
+		(property "LCSC Part" "C475624"
+			(at 237.49 114.3 0)
+			(effects
+				(font
+					(size 1.27 1.27)
+				)
+				(hide yes)
+			)
+		)
+		(pin "1"
+		)
+		(pin "2"
+		)
+		(instances
+			(project ""
+				(path "/b3a59d80-e104-4a02-9d1b-dc2012df0476"
+					(reference "D2")
+					(unit 1)
+				)

Commit message: Production pcb ordered to jlcpcb
Parts:
- J1: value G14A421211112HR -> G14A42121B12HR; footprint amphenol_oculink:AMPHENOL_G14A421211112HR -> amphenol_oculink:AMPHENOL_G14A42121B12HR; symbol G14A421211112HR:G14A421211112HR -> G14A42121B12HR:G14A42121B12HR; MAXIMUM_PACKAGE_HEIGHT 3.92mm -> 3.9mm; PARTREV A -> D
Changed lines of the file:
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@@
 	)
 	(symbol
-		(lib_id "G14A421211112HR:G14A421211112HR")
-		(at 186.69 111.76 0)
+		(lib_id "G14A42121B12HR:G14A42121B12HR")
+		(at 186.69 113.03 0)
 		(unit 1)
 		(exclude_from_sim no)
@@
 			)
 		)
-		(property "Value" "G14A421211112HR"
+		(property "Value" "G14A42121B12HR"
 			(at 186.69 78.74 0)
 			(effects
@@
 			)
 		)
-		(property "Footprint" "amphenol_oculink:AMPHENOL_G14A421211112HR"
-			(at 186.436 67.818 0)
+		(property "Footprint" "amphenol_oculink:AMPHENOL_G14A42121B12HR"
+			(at 187.96 69.85 0)
 			(effects
 				(font
@@
 		)
 		(property "Datasheet" ""
-			(at 186.69 111.76 0)
+			(at 185.42 113.03 0)
 			(effects
 				(font
@@
 		)
 		(property "Description" ""
-			(at 186.69 111.76 0)
+			(at 185.42 113.03 0)
 			(effects
 				(font
@@
 			)
 		)
-		(property "PARTREV" "A"
-			(at 186.69 64.516 0)
+		(property "PARTREV" "D"
+			(at 186.69 67.31 0)
 			(effects
 				(font
@@
 		)
 		(property "STANDARD" "Manufacturer Recommendations"
-			(at 186.944 70.358 0)
+			(at 188.468 72.39 0)
 			(effects
 				(font
@@
 			)
 		)
-		(property "MAXIMUM_PACKAGE_HEIGHT" "3.92mm"
-			(at 186.944 72.898 0)
+		(property "MAXIMUM_PACKAGE_HEIGHT" "3.9mm"
+			(at 186.182 78.232 0)
 			(effects
 				(font
@@
 		)
 		(property "MANUFACTURER" "Amphenol"
-			(at 186.944 74.93 0)
+			(at 186.944 75.184 0)
 			(effects
 				(font
@@
 		)
 		(property "LCSC Part" "C5156927"
-			(at 186.69 111.76 0)
+			(at 186.69 113.03 0)
 			(effects
 				(font
