File: kicad/oculink_m2.kicad_pcb (KiCad board)
At the start: 4 copper layers, 99.5 x 58 mm, 13 parts, among them J1 G14A42121B12HR

Commit message: Improved ground stitching and fix skew on clock differential pair
Parts:
- moved TP1 0.22 mm to (118.5, 49.6)
Routing:
- net TX0-: track 132.6 -> 131.4 mm
- net TX0+: track 132.6 -> 131.4 mm
- net CLOCK-: track 149.5 -> 150.5 mm
- net CLKREQ: track 160.4 -> 161.1 mm
- net SMB-: track 163.0 -> 162.5 mm
- net SMB+: track 163.0 -> 162.5 mm
- net PERST: track 161.6 -> 162.1 mm
- net GND: vias 1335 -> 1363

Commit message: Swapped SMB pair to connect clock/data correctly
Parts:
- J1: value G14A42121B12HR -> G14A421211112HR
Connections:
- J1 pad B10: SMB- -> SMB+
- J1 pad B9: SMB+ -> SMB-
Routing:
- net SMB-: track 162.5 -> 160.5 mm
- net SMB+: track 162.5 -> 161.5 mm
- net GND: vias 1363 -> 1374

Commit message: Added additional mounting holes for adapter
Parts:
- added D1: Power LED, LED_SMD:LED_1206_3216Metric_Pad1.42x1.75mm_HandSolder, B.Cu at (193.2, 98.6)
- added H2: MOUNT_1, MountingHole:MountingHole_2.7mm, F.Cu at (182.7, 71.0)
- added H3: MOUNT_2, MountingHole:MountingHole_2.7mm, F.Cu at (188.3, 147.7)
- added R1: 100, Resistor_SMD:R_0603_1608Metric, B.Cu at (188.6, 98.6)
- moved J1 8.27 mm to (190.0, 85.3)
- moved C1 8.20 mm to (99.4, 60.8)
- moved C4 8.20 mm to (96.9, 41.4)
- moved E1 8.20 mm to (109.5, 51.0)
- moved H1 8.20 mm to (133.0, 51.0)
- moved TP1 8.20 mm to (118.5, 41.4)
- moved C5 8.20 mm to (95.2, 53.1)
- moved JP1 8.20 mm to (100.4, 35.5)
- moved JP3 8.20 mm to (110.8, 35.5)
- moved C2 7.34 mm to (179.3, 94.6)
- moved C3 6.93 mm to (181.5, 94.6)
- moved TP9 6.15 mm to (184.8, 98.6)
- moved JP2 5.70 mm to (180.1, 98.7)
Routing:
- net GND: track 944.1 -> 965.6 mm, vias 1374 -> 1493
- net 3.3V_OPT: track 11.8 -> 21.0 mm, vias 1 -> 2
- net Net-(D1-A): track 0.00 -> 4.87 mm
- net RX0-: track 137.6 -> 142.0 mm
- net TX0-: track 131.4 -> 135.8 mm
- net TX0+: track 131.4 -> 135.8 mm
- net RX0+: track 137.6 -> 142.0 mm
- net RX1+: track 137.5 -> 141.9 mm
- net RX1-: track 137.5 -> 141.9 mm
- net TX1-: track 132.4 -> 136.4 mm
- net TX1+: track 132.4 -> 136.4 mm
- net CLOCK-: track 150.5 -> 146.6 mm
- net CLOCK+: track 150.5 -> 146.6 mm
- net SMB+: track 161.5 -> 158.5 mm
- net SMB-: track 160.5 -> 158.5 mm
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Other:
- board size 99.5 x 58 mm -> 100.5 x 112.3 mm

Commit message: Fixed position of additional mounting holes and made them oval vertically for potential vertical adjustment of adapter
Parts:
- moved H3 1.00 mm to (187.5, 147.1)
- moved H2 0.65 mm to (182.7, 70.3)
Routing:
- net GND: track 965.6 -> 965.8 mm, vias 1493 -> 1492
Other:
- board size 100.5 x 112.3 mm -> 100.5 x 113.2 mm

Commit message: Fixed ground pour overflowing onto m2 edge connector
Routing:
- net GND: vias 1492 -> 1491
Changed lines of the file:
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@@
 	)
 	(via
-		(at 189 101.8)
-		(size 0.35)
-		(drill 0.2)
-		(layers "F.Cu" "B.Cu")
-		(free yes)
-		(net 1)
-	)
-	(via
 		(at 126 52.8)
 		(size 0.35)
@@
 		(polygon
 			(pts
-				(xy 93.025 38.95) (xy 199.325 39) (xy 199.325 103.75) (xy 93.025 103.7)
+				(xy 93.275 38.95) (xy 199.375 39) (xy 199.375 103.75) (xy 93.275 103.7)
 			)
 		)

Commit message: Added stackup information to schematic
Other:
- board text added: "0"
- board text added: "0 mm"
- board text added: "0.0152 mm"
- board text added: "0.01524 mm"
- board text added: "0.02"
- board text added: "0.035 mm"
- board text added: "0.0900 mm / 0.0900 mm"
- board text added: "0.0994 mm"
- board text added: "0.1500 mm"
- board text added: "0.45 mm"
- board text added: "0.7797 mm"
- board text added: "1"
- board text added: "104.7250 mm x 113.2111 mm"
- board text added: "3.8"
- board text added: "3113x1"
- board text added: "4"
- board text added: "4.1"
- board text added: "4.6"
- board text added: "B.Cu"
- board text added: "B.Mask"
- board text added: "B.Paste"
- board text added: "B.Silkscreen"
- board text added: "BOARD CHARACTERISTICS"
- board text added: "Board Thickness:"
- board text added: "Board overall dimensions:"
- board text added: "Bottom Silk Screen"
- board text added: "Bottom Solder Mask"
- board text added: "Bottom Solder Paste"
- board text added: "Castellated pads:"
- board text added: "Color"
- board text added: "Copper Finish:"
- board text added: "Copper Layer Count:"
- board text added: "Core"
- board text added: "Dielectric 1"
- board text added: "Dielectric 2"
- board text added: "Dielectric 3"
- board text added: "Direct Printing"
- board text added: "Edge card connectors:"
- board text added: "Epsilon R"
- board text added: "F.Cu"
- board text added: "F.Mask"
- board text added: "F.Paste"
- board text added: "F.Silkscreen"
- board text added: "FR4 natural"
- board text added: "Green"
- board text added: "Impedance Control:"
- board text added: "In1.Cu"
- board text added: "In2.Cu"
- board text added: "Layer Name"
- board text added: "Loss Tangent"
- board text added: "Material"
- board text added: "Min hole diameter:"
- board text added: "Min track/spacing:"
- board text added: "No"
- board text added: "None"
- board text added: "Not specified"
- board text added: "PCIE 4.0 x 4 M2 to Oculink Adapter for 16ARP8 Laptop"
- board text added: "Plated Board Edge:"
- board text added: "Thickness (mm)"
- board text added: "Top Silk Screen"
- board text added: "Top Solder Mask"
- board text added: "Top Solder Paste"
- board text added: "Type"
- board text added: "White"
- board text added: "Yes"
- board text added: "copper"
- board text added: "core"
- board text added: "prepreg"

Commit message: Fixed mounting holes
Parts:
- H2, H3: footprint MountingHole:MountingHole_2.7mm -> custom_edge_connector:secondary_mounting_hole
- moved H3 5.05 mm to (187.5, 142.1)
- moved H2 5.00 mm to (182.7, 65.3)
