File: kicad/oculink_m2.kicad_pcb (KiCad board)
At the start: 4 copper layers, 100.5 x 113.2 mm, 17 parts, among them J1 G14A421211112HR

Commit message: Updated bom script and added in schottky diode on clkreq
Parts:
- added D2: D_Schottky, Diode_SMD:D_SOD-523, B.Cu at (104.4, 43.3)
- moved JP1 0.50 mm to (100.4, 35.0)
- moved JP3 0.50 mm to (110.8, 35.0)
Connections:
- J1 pad B13: CLKREQ -> /CLKREQ_EXT
Routing:
- net CLKREQ: track 160.5 -> 13.1 mm, vias 2 -> 0
- net /CLKREQ_EXT: track 0.00 -> 146.7 mm, vias 0 -> 2
- net GND: vias 1491 -> 1496

Commit message: Production pcb ordered to jlcpcb
Parts:
- J1: value G14A421211112HR -> G14A42121B12HR; footprint amphenol_oculink:AMPHENOL_G14A421211112HR -> amphenol_oculink:AMPHENOL_G14A42121B12HR
Routing:
- net GND: vias 1496 -> 1457
Other:
- board text added: "PCIE 4.0 x 4 M2 to Oculink Adapter for Lenovo 16ARP8 Laptop Revision 1.0 William Yang 2024"
