File: kicad/oculink_m2.kicad_pcb (KiCad board)
At the start: 4 copper layers, 100.5 x 113.2 mm, 18 parts, among them J1 G14A42121B12HR

Commit message: Added design rule check for 85ohm impedance matched differential pairs
Routing:
- net SMB-: track 158.5 -> 157.6 mm

Commit message: Fixed up diff pair custom rules
Routing:
- net SMB-: track 157.6 -> 158.5 mm

Commit message: Updated design rules to allow for denser via fence
Routing:
- net /PEWAKE_EXT: track 172.1 -> 172.9 mm
- net /CLKREQ_EXT: track 146.7 -> 146.0 mm
- net /PEDET_EXT: track 172.0 -> 172.6 mm
- net GND: vias 1457 -> 1420

Commit message: Start of dense via layout
Parts:
- moved C5 1.20 mm to (96.4, 53.1), turned to 0 degrees
Routing:
- net GND: track 965.8 -> 931.3 mm, vias 1420 -> 810
- net /PEWAKE_EXT: track 172.9 -> 174.1 mm, vias 5 -> 4
- net +3.3V: track 165.6 -> 164.7 mm

Commit message: Applied vias to half of board
Routing:
- net GND: track 931.3 -> 957.3 mm, vias 810 -> 2447
- net /PEWAKE_EXT: track 174.1 -> 172.9 mm
- net PEWAKE: track 20.3 -> 21.1 mm

Commit message: Finished right angle section
Routing:
- net RX0-: track 142.0 -> 138.8 mm
- net RX0+: track 142.0 -> 138.8 mm
- net /PEWAKE_EXT: track 172.9 -> 174.1 mm, vias 4 -> 5
- net TX0-: track 135.8 -> 134.7 mm
- net TX0+: track 135.8 -> 134.7 mm
- net GND: track 957.3 -> 956.4 mm, vias 2447 -> 2974
- net /PEDET_EXT: track 172.8 -> 173.5 mm

Commit message: Finished applying vias to connector section
Routing:
- net GND: track 956.4 -> 956.0 mm, vias 2974 -> 3421
