File: kicad/oculink_m2_flex_connector/oculink_port/oculink_port.kicad_pcb (KiCad board)
At the start: 4 copper layers, 20.8 x 32.9 mm, 8 parts, among them J1 G14A42121B12HR, J2 Conn_01x38_Pin

Commit message: Initial layout of port side board
Parts:
- removed H1, H2: MountingHole_Pad, custom:mounting_pad_1mm
- J2: moved to B.Cu
- moved C5 6.93 mm to (146.9, 106.9), turned to -90 degrees
- moved C1 6.37 mm to (142.2, 106.9), turned to -90 degrees
- moved TP2 3.17 mm to (153.6, 105.3)
- moved J2 1.70 mm to (138.8, 80.4), turned to 180 degrees
- moved J1 1.21 mm to (151.0, 92.5)
- moved JP1 0.90 mm to (144.6, 104.1), turned to 0 degrees
Connections:
- J2 pad 14: SMB- -> RX1+
- J2 pad 15: SMB+ -> RX1-
- J2 pad 17: PERST -> TX2+
- J2 pad 18: CLKREQ -> TX2-
- J2 pad 19: PEDET -> GND
- J2 pad 2: RX1- -> CLOCK+
- J2 pad 20: PEWAKE -> RX2+
- J2 pad 21: GND -> RX2-
- J2 pad 22: CLOCK+ -> GND
- J2 pad 23: CLOCK- -> TX3+
- J2 pad 24: GND -> TX3-
- J2 pad 25: TX2+ -> GND
- J2 pad 26: TX2- -> RX3+
- J2 pad 27: GND -> RX3-
- J2 pad 28: TX3+ -> GND
- J2 pad 29: TX3- -> CLKREQ
- J2 pad 3: RX1+ -> CLOCK-
- J2 pad 30: GND -> PERST
- J2 pad 31: RX3- -> PEWAKE
- J2 pad 32: RX3+ -> PEDET
- J2 pad 33: GND -> 3.3V_OPT
- J2 pad 34: RX2- -> GND
- J2 pad 5: RX0- -> TX0+
- J2 pad 6: RX0+ -> TX0-
- J2 pad 8: TX0+ -> RX0+
- J2 pad 9: TX0- -> RX0-
Routing:
- net CLKREQ: track 9.98 -> 32.5 mm, vias 0 -> 3
- net PERST: track 10.0 -> 31.4 mm, vias 0 -> 1
- net 3.3V: track 30.4 -> 11.7 mm, vias 2 -> 0
- net CLOCK-: track 20.7 -> 33.7 mm, vias 2 -> 1
- net RX2+: track 26.4 -> 15.4 mm, vias 0 -> 1
- net PEDET: track 20.4 -> 31.2 mm, vias 2 -> 3
- net CLOCK+: track 20.7 -> 31.0 mm, vias 2 -> 1
- net SMB+: track 9.55 -> 0.00 mm
- net SMB-: track 9.55 -> 0.00 mm
- net RX2-: track 24.9 -> 15.4 mm, vias 0 -> 1
- net RX1-: track 27.5 -> 18.4 mm, vias 0 -> 1
- net RX1+: track 26.0 -> 18.4 mm, vias 0 -> 1
- net PEWAKE: track 21.4 -> 29.0 mm, vias 2 -> 1
- net RX0-: track 22.2 -> 15.3 mm, vias 0 -> 1
- net RX0+: track 20.7 -> 15.3 mm, vias 0 -> 1
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Other:
- board text removed: "JLC04161H-2116D Stackup"

Commit message: Set correct impedance on port pcb
Routing:
- net RX3-: track 20.4 -> 18.4 mm, vias 2 -> 1
- net RX3+: track 20.4 -> 18.4 mm, vias 2 -> 1
- net CLOCK+: track 31.0 -> 32.0 mm
- net CLOCK-: track 33.7 -> 34.4 mm
- net 3.3V: track 11.7 -> 12.3 mm
- net GND: vias 223 -> 215

Commit message: Added mounting for port
Parts:
- added ?: , , F.Cu at (187.1, 68.8)
- added ?: , , F.Cu at (192.2, 145.6)
- moved C1 46.3 mm to (186.3, 121.0)
- moved C5 46.3 mm to (191.0, 121.0)
- moved J1 46.3 mm to (195.1, 106.6)
- moved J2 46.3 mm to (182.8, 94.5)
- moved JP1 46.3 mm to (188.7, 118.2)
- moved TP2 42.9 mm to (194.2, 119.2)
Routing:
- net 3.3V_OPT: track 11.7 -> 12.3 mm
- net GND: vias 215 -> 205
Other:
- board size 20.8 x 32.9 mm -> 20.7 x 87.1 mm

Commit message: Shifted location of ffc connector to avoid screw mount
Parts:
- moved J2 4.50 mm to (182.9, 99.0)
- moved JP1 0.95 mm to (189.0, 119.1)
- moved J1 0.61 mm to (195.7, 106.6)
- moved C5 0.40 mm to (191.4, 121.0)
- moved TP2 0.32 mm to (194.5, 119.2)
- moved C1 0.32 mm to (186.6, 121.0)
Routing:
- net CLOCK+: track 32.0 -> 37.6 mm
- net CLOCK-: track 34.4 -> 40.1 mm
- net RX1-: track 18.4 -> 23.7 mm
- net RX1+: track 18.4 -> 23.7 mm
- net TX1-: track 9.73 -> 14.0 mm
- net TX1+: track 9.73 -> 14.0 mm
- net RX0+: track 15.3 -> 19.5 mm
- net RX0-: track 15.3 -> 19.5 mm
- net RX3-: track 18.4 -> 22.3 mm
- net RX3+: track 18.4 -> 22.3 mm
- net TX3+: track 9.73 -> 13.4 mm
- net TX3-: track 9.73 -> 13.4 mm
- net PERST: track 31.4 -> 34.8 mm
- net TX0-: track 9.93 -> 12.7 mm
- net TX0+: track 9.95 -> 12.7 mm
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