File: kicad/oculink_m2_flex_connector/flex_pcb/flex_pcb.kicad_sch (KiCad schematic)
At the start: 3 parts, among them J1 Conn_02x01, J2 Conn_02x01

Commit message: Crude flex pcb layout
Parts:
- removed J1, J2: Conn_02x01, Connector_Samtec_MicroPower:Samtec_UMPS-02-XX.X-X-V-S_1x02_P2.0mm_Socket, symbol Connector_Generic:Conn_02x01
- removed TP1: TestPoint, TestPoint:TestPoint_Pad_D1.0mm, symbol Connector:TestPoint
- added J1, J2: Conn_01x38_Pin, flex_connector:port_pcb, symbol Connector:Conn_01x34_Pin
Connections:
- net GND: now also J1.1 (Pin_1), J1.10 (Pin_10), J1.13 (Pin_13), J1.16 (Pin_16), J1.19 (Pin_19), J1.22 (Pin_22), J1.25 (Pin_25), J1.28 (Pin_28), J1.34 (Pin_34), J1.4 (Pin_4), J1.7 (Pin_7), J2.1 (Pin_1), J2.10 (Pin_10), J2.13 (Pin_13), J2.16 (Pin_16), J2.19 (Pin_19), J2.22 (Pin_22), J2.25 (Pin_25), J2.28 (Pin_28), J2.34 (Pin_34), J2.4 (Pin_4), J2.7 (Pin_7)
- new net 3.3V_OPT: J1.33 (Pin_33), J2.33 (Pin_33)
- new net CLKREQ: J1.29 (Pin_29), J2.29 (Pin_29)
- new net CLOCK+: J1.2 (Pin_2), J2.2 (Pin_2)
- new net CLOCK-: J1.3 (Pin_3), J2.3 (Pin_3)
- new net PEDET: J1.32 (Pin_32), J2.32 (Pin_32)
- new net PERST: J1.30 (Pin_30), J2.30 (Pin_30)
- new net PEWAKE: J1.31 (Pin_31), J2.31 (Pin_31)
- new net RX0+: J1.8 (Pin_8), J2.8 (Pin_8)
- new net RX0-: J1.9 (Pin_9), J2.9 (Pin_9)
- new net RX1+: J1.14 (Pin_14), J2.14 (Pin_14)
- new net RX1-: J1.15 (Pin_15), J2.15 (Pin_15)
- new net RX2+: J1.20 (Pin_20), J2.20 (Pin_20)
- new net RX2-: J1.21 (Pin_21), J2.21 (Pin_21)
- new net RX3+: J1.26 (Pin_26), J2.26 (Pin_26)
- new net RX3-: J1.27 (Pin_27), J2.27 (Pin_27)
- new net TX0+: J1.5 (Pin_5), J2.5 (Pin_5)
- new net TX0-: J1.6 (Pin_6), J2.6 (Pin_6)
- new net TX1+: J1.11 (Pin_11), J2.11 (Pin_11)
- new net TX1-: J1.12 (Pin_12), J2.12 (Pin_12)
- new net TX2+: J1.17 (Pin_17), J2.17 (Pin_17)
- new net TX2-: J1.18 (Pin_18), J2.18 (Pin_18)
- new net TX3+: J1.23 (Pin_23), J2.23 (Pin_23)
- new net TX3-: J1.24 (Pin_24), J2.24 (Pin_24)
