File: kicad/oculink_m2_flex_connector/flex_pcb/flex_pcb.kicad_pcb (KiCad board)
At the start: 2 copper layers, 42 x 20 mm, 3 parts, among them J1 Conn_02x01, J2 Conn_02x01

Commit message: Crude flex pcb layout
Parts:
- removed TP1: TestPoint, TestPoint:TestPoint_Pad_D1.0mm
- J1, J2: value Conn_02x01 -> Conn_01x38_Pin; footprint Connector_Samtec_MicroPower:Samtec_UMPS-02-XX.X-X-V-S_1x02_P2.0mm_Socket -> flex_connector:port_pcb
- moved J2 17.4 mm to (117.6, 66.8), turned to 0 degrees
- moved J1 13.2 mm to (94.0, 66.8), turned to 0 degrees
Connections:
- net D- renamed CLOCK+
- J1 pad 1: D+ -> GND
- J2 pad 1: D+ -> GND
Routing:
- net GND: track 0.00 -> 259.6 mm, vias 0 -> 396
- net D+: track 36.6 -> 0.00 mm
- net TX3-: track 0.00 -> 23.6 mm
- net TX3+: track 0.00 -> 23.6 mm
- net TX2-: track 0.00 -> 23.6 mm
- net TX2+: track 0.00 -> 23.6 mm
- net TX1-: track 0.00 -> 23.6 mm
- net TX1+: track 0.00 -> 23.6 mm
- net TX0-: track 0.00 -> 23.6 mm
- net TX0+: track 0.00 -> 23.6 mm
- net RX3-: track 0.00 -> 23.6 mm
- net RX3+: track 0.00 -> 23.6 mm
- net RX2-: track 0.00 -> 23.6 mm
- net RX2+: track 0.00 -> 23.6 mm
- net RX1-: track 0.00 -> 23.6 mm
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- added copper zone on F.Cu, net GND
Other:
- board size 42 x 20 mm -> 29.7 x 17.5 mm

Commit message: Test design for consistent hatched ground plane
Routing:
- net GND: track 259.6 -> 569.0 mm
Other:
- board size 29.7 x 17.5 mm -> 29.7 x 17.8 mm

Commit message: Unified taper geometry across pcbs
Routing:
- net GND: track 569.0 -> 512.9 mm
Changed lines of the file:
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@@
-	)
-	(segment
-		(start 117.1 85.2)
-		(end 119.85 85.2)
-		(width 0.5)
-		(layer "F.Cu")
-		(net 1)
-	)
-	(segment
-		(start 94.3 74.7)
-		(end 91.75 74.7)
-		(width 0.5)
-		(layer "F.Cu")
-		(net 1)
 	)
 	(segment
 		(start 97 71.7)
 		(end 94.25 71.7)
-		(width 0.5)
-		(layer "F.Cu")
-		(net 1)
-	)
-	(segment
-		(start 117.2 79.2)
-		(end 119.85 79.2)
 		(width 0.5)
 		(layer "F.Cu")
@@
 	)
 	(segment
-		(start 94.2 83.7)
-		(end 91.75 83.7)
-		(width 0.5)
-		(layer "F.Cu")
-		(net 1)
-	)
-	(segment
-		(start 117.2 82.2)
-		(end 119.85 82.2)
-		(width 0.5)
-		(layer "F.Cu")
-		(net 1)
-	)
-	(segment
 		(start 97 80.7)
 		(end 94.2 80.7)
-		(width 0.5)
-		(layer "F.Cu")
-		(net 1)
-	)
-	(segment
-		(start 117.2 76.2)
-		(end 119.55 76.2)
-		(width 0.5)
-		(layer "F.Cu")
-		(net 1)
-	)
-	(segment
-		(start 94.25 71.7)
-		(end 91.75 71.7)
-		(width 0.5)
-		(layer "F.Cu")
-		(net 1)
-	)
-	(segment
-		(start 94.3 76.2)
-		(end 91.75 76.2)
 		(width 0.5)
 		(layer "F.Cu")
@@
 	)
 	(segment
-		(start 117.2 77.7)
-		(end 119.85 77.7)
-		(width 0.5)
-		(layer "F.Cu")
-		(net 1)
-	)
-	(segment
 		(start 114.5 79.2)
 		(end 117.2 79.2)
-		(width 0.5)
-		(layer "F.Cu")
-		(net 1)
-	)
-	(segment
-		(start 94.2 79.2)
-		(end 91.75 79.2)
-		(width 0.5)
-		(layer "F.Cu")
-		(net 1)
-	)
-	(segment
-		(start 94.25 73.2)
-		(end 91.75 73.2)
 		(width 0.5)
 		(layer "F.Cu")
@@
 	)
 	(segment
-		(start 117.2 80.7)
-		(end 119.85 80.7)
-		(width 0.5)
-		(layer "F.Cu")
-		(net 1)
-	)
-	(segment
 		(start 114.5 76.2)
 		(end 117.2 76.2)
-		(width 0.5)
-		(layer "F.Cu")
-		(net 1)
-	)
-	(segment
-		(start 117.175 73.2)
-		(end 119.85 73.2)
 		(width 0.5)
 		(layer "F.Cu")
@@
 	)
 	(segment
-		(start 117.25 71.7)
-		(end 119.85 71.7)
-		(width 0.5)
-		(layer "F.Cu")
-		(net 1)
-	)
-	(segment
-		(start 117.2 74.7)
-		(end 119.85 74.7)
-		(width 0.5)
-		(layer "F.Cu")
-		(net 1)
-	)
-	(segment
 		(start 97 87.95)
 		(end 117.1 87.95)
@@
 		(start 97 71.7)
 		(end 117.25 71.7)
-		(width 0.5)
-		(layer "F.Cu")
-		(net 1)
-	)
-	(segment
-		(start 94.1 85.2)
-		(end 91.75 85.2)
-		(width 0.5)
-		(layer "F.Cu")
-		(net 1)
-	)
-	(segment
-		(start 117.1 83.7)
-		(end 119.85 83.7)
-		(width 0.5)
-		(layer "F.Cu")
-		(net 1)
-	)
-	(segment
-		(start 94.2 80.7)
-		(end 91.75 80.7)
-		(width 0.5)
-		(layer "F.Cu")
-		(net 1)
-	)
-	(segment
-		(start 94.1 87.95)
-		(end 91.75 87.95)
-		(width 0.5)
-		(layer "F.Cu")
-		(net 1)
-	)
-	(segment
-		(start 117.1 87.95)
-		(end 119.85 87.95)
-		(width 0.5)
-		(layer "F.Cu")
-		(net 1)
-	)
-	(segment
-		(start 94.2 77.7)
-		(end 91.75 77.7)
 		(width 0.5)
 		(layer "F.Cu")
@@
 		(width 0.5)
 		(layer "F.Cu")
-		(net 1)
-	)
-	(segment
-		(start 94.2 82.2)
-		(end 91.75 82.2)
-		(width 0.5)
-		(layer "F.Cu")

Commit message: Added taper for ground ffc pads
Routing:
- net GND: track 512.9 -> 517.7 mm

Commit message: Initial design and layout for flex pcb
Parts:
- moved J2 78.5 mm to (170.1, 125.3)
- moved J1 1.69 mm to (92.8, 65.7)
Routing:
- net GND: track 517.7 -> 2654.9 mm, vias 396 -> 692
- net 3.3V_OPT: track 23.6 -> 120.7 mm
- net PERST: track 23.6 -> 120.7 mm
- net PEWAKE: track 23.6 -> 120.7 mm
- net PEDET: track 23.6 -> 120.7 mm
- net RX3-: track 23.6 -> 120.7 mm
- net CLKREQ: track 23.6 -> 120.7 mm
- net RX3+: track 23.6 -> 120.7 mm
- net TX1+: track 23.6 -> 120.7 mm
- net RX1-: track 23.6 -> 120.7 mm
- net TX1-: track 23.6 -> 120.7 mm
- net RX1+: track 23.6 -> 120.7 mm
- net TX0-: track 23.6 -> 120.7 mm
- net TX0+: track 23.6 -> 120.7 mm
- net RX2+: track 23.6 -> 120.7 mm
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- removed copper zone on F.Cu, net GND
Other:
- board size 29.7 x 17.8 mm -> 82.9 x 76.9 mm

Commit message: Finished initial layout of hatched plane for differential traces
Routing:
- added copper zone on F.Cu, net GND

Commit message: Finished via fencing on flex pcb
Routing:
- net GND: vias 692 -> 2143
