File: simulations/differential_taper/differential.kicad_pcb (KiCad board)
At the start: 4 copper layers, 1.3 x 2.1 mm, 5 parts

Commit message: Updated taper simulation
Parts:
- moved SP0 2.15 mm to (148.5, 125.3)
- moved SP2 2.15 mm to (148.8, 125.3)
- moved GND1 2.07 mm to (148.4, 125.0)
Routing:
- net A-: track 1.03 -> 3.18 mm
- net A+: track 1.03 -> 3.18 mm
- net GND: vias 6 -> 40
Other:
- board size 1.3 x 2.1 mm -> 1.3 x 4.2 mm
