File: simulations/differential_hatched/differential.kicad_sch (KiCad schematic)
At the start: 5 parts

Commit message: Updated trace width to 0.15mm instead of 0.1mm
Parts:
- SP0, SP1, SP2, SP3: footprint simulation_port:pad_0.1mm -> simulation_port:pad_0.15mm
Changed lines of the file:
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@@
 			)
 		)
-		(property "Footprint" "simulation_port:pad_0.1mm"
+		(property "Footprint" "simulation_port:pad_0.15mm"
 			(at 118.11 71.12 0)
 			(effects
@@
 			)
 		)
-		(property "Footprint" "simulation_port:pad_0.1mm"
+		(property "Footprint" "simulation_port:pad_0.15mm"
 			(at 107.95 134.62 0)
 			(effects
@@
 			)
 		)
-		(property "Footprint" "simulation_port:pad_0.1mm"
+		(property "Footprint" "simulation_port:pad_0.15mm"
 			(at 144.78 71.12 0)
 			(effects
@@
 			)
 		)
-		(property "Footprint" "simulation_port:pad_0.1mm"
+		(property "Footprint" "simulation_port:pad_0.15mm"
 			(at 134.62 134.62 0)
 			(effects
